File: v1/pcbs/cornish.kicad_pcb (KiCad board)
At the start: 2 copper layers, 155.9 x 133.8 mm, 50 parts

Commit message: v1.0
Parts:
- removed MCU1: , ProMicro
- removed _1, _2, _3, _4, _5, _6: , MountingHole_2.2mm_M2_Pad_Via
- added REF**: VIA-0.6mm, VIA-0.6mm, F.Cu at (140.5, 125.6)
- added REF**: VIA-0.6mm, VIA-0.6mm, F.Cu at (197.8, 139.0)
- added REF**: VIA-0.6mm, VIA-0.6mm, F.Cu at (205.8, 121.8)
- added REF**: VIA-0.6mm, VIA-0.6mm, F.Cu at (213.8, 104.6)
- added REF**: VIA-0.6mm, VIA-0.6mm, F.Cu at (215.0, 147.0)
- added REF**: VIA-0.6mm, VIA-0.6mm, F.Cu at (223.0, 129.8)
- added REF**: VIA-0.6mm, VIA-0.6mm, F.Cu at (231.1, 112.6)
- added REF**: VIA-0.6mm, VIA-0.6mm, F.Cu at (192.7, 160.9)
- added REF**: VIA-0.6mm, VIA-0.6mm, F.Cu at (216.1, 173.8)
- added REF**: VIA-0.6mm, VIA-0.6mm, F.Cu at (234.8, 193.3)
- added REF**: VIA-0.6mm, VIA-0.6mm, F.Cu at (238.9, 152.7)
- added REF**: VIA-0.6mm, VIA-0.6mm, F.Cu at (147.0, 107.8)
- added REF**: VIA-0.6mm, VIA-0.6mm, F.Cu at (246.9, 135.4)
- added REF**: VIA-0.6mm, VIA-0.6mm, F.Cu at (149.9, 129.1)
- added REF**: VIA-0.6mm, VIA-0.6mm, F.Cu at (156.4, 111.2)
- added REF**: VIA-0.6mm, VIA-0.6mm, F.Cu at (162.9, 93.3)
- added REF**: VIA-0.6mm, VIA-0.6mm, F.Cu at (172.8, 126.3)
- added REF**: VIA-0.6mm, VIA-0.6mm, F.Cu at (180.9, 109.1)
- added REF**: VIA-0.6mm, VIA-0.6mm, F.Cu at (188.9, 91.8)
- added REF**: VIA-0.6mm, VIA-0.6mm, F.Cu at (192.2, 129.8)
- added REF**: VIA-0.6mm, VIA-0.6mm, F.Cu at (200.2, 112.6)
- added REF**: VIA-0.6mm, VIA-0.6mm, F.Cu at (208.2, 95.3)
- added REF**: VIA-0.6mm, VIA-0.6mm, F.Cu at (153.5, 89.9)
- added REF**: VIA-0.6mm, VIA-0.6mm, F.Cu at (206.8, 143.2)
- added REF**: VIA-0.6mm, VIA-0.6mm, F.Cu at (214.9, 126.0)
- added REF**: VIA-0.6mm, VIA-0.6mm, F.Cu at (222.9, 108.8)
- added REF**: VIA-0.6mm, VIA-0.6mm, F.Cu at (224.1, 151.3)
- added REF**: VIA-0.6mm, VIA-0.6mm, F.Cu at (232.1, 134.1)
- added REF**: VIA-0.6mm, VIA-0.6mm, F.Cu at (240.1, 116.8)
- added REF**: VIA-0.6mm, VIA-0.6mm, F.Cu at (201.8, 165.2)
- added REF**: VIA-0.6mm, VIA-0.6mm, F.Cu at (223.8, 180.2)
- added REF**: VIA-0.6mm, VIA-0.6mm, F.Cu at (243.0, 187.6)
- added REF**: VIA-0.6mm, VIA-0.6mm, F.Cu at (247.9, 156.9)
- added REF**: VIA-0.6mm, VIA-0.6mm, F.Cu at (163.8, 122.1)
- added REF**: VIA-0.6mm, VIA-0.6mm, F.Cu at (256.0, 139.7)
- added REF**: VIA-0.6mm, VIA-0.6mm, F.Cu at (171.8, 104.8)
- added REF**: VIA-0.6mm, VIA-0.6mm, F.Cu at (179.8, 87.6)
- added REF**: VIA-0.6mm, VIA-0.6mm, F.Cu at (183.1, 125.6)
- added REF**: VIA-0.6mm, VIA-0.6mm, F.Cu at (191.1, 108.3)
- added REF**: VIA-0.6mm, VIA-0.6mm, F.Cu at (199.2, 91.1)
- added _41: , ProMicro, F.Cu at (269.3, 153.6)
- added _42: , MountingHole_2.2mm_M2_Pad_Via, F.Cu at (170.0, 92.7)
- added _43: , MountingHole_2.2mm_M2_Pad_Via, F.Cu at (155.8, 121.6)
- added _44: , MountingHole_2.2mm_M2_Pad_Via, F.Cu at (205.7, 111.3)
- added _45: , MountingHole_2.2mm_M2_Pad_Via, F.Cu at (190.9, 149.6)
- added _46: , MountingHole_2.2mm_M2_Pad_Via, F.Cu at (258.0, 123.5)
- added _47: , MountingHole_2.2mm_M2_Pad_Via, F.Cu at (239.1, 171.0)
- S1, S10, S11, S12, S13, S14, S15, S16, S17, S18, S19, S2, S20, S3, S4, S5, S6, S7, S8, S9: value MXLP -> ks33; footprint MX-Low-Profile -> Gateron-Low-Profile-ks-33
- moved D18 10.00 mm to (236.1, 186.3)
- moved D1 10.00 mm to (146.9, 122.6)
- moved D2 10.00 mm to (153.4, 104.8)
- moved D3 10.00 mm to (159.9, 86.9)
- moved D11 10.00 mm to (212.5, 119.4)
- moved D12 10.00 mm to (220.5, 102.2)
- moved D15 10.00 mm to (237.7, 110.2)
- moved D5 10.00 mm to (178.4, 102.4)
- moved D6 10.00 mm to (186.5, 85.2)
- moved D7 10.00 mm to (189.7, 123.1)
- moved D8 10.00 mm to (197.8, 105.9)
- moved D9 10.00 mm to (205.8, 88.7)
- moved D14 10.00 mm to (229.7, 127.4)
- moved D4 10.00 mm to (170.4, 119.6)
- moved D10 10.00 mm to (204.4, 136.6)
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
Commit message: v1.1 and case
Parts:
- moved TRRS1 2.00 mm to (254.8, 113.7)
- moved B1 1.00 mm to (258.7, 176.3)
- moved _41 1.00 mm to (268.9, 154.5)
- moved OLED1 1.00 mm to (267.8, 171.1)
Other:
- board size 155.9 x 133.8 mm -> 152.8 x 129.3 mm
